Commit message: Adding tcp to ball joint and model comparison.

File: assets/panda.urdf (robot description, URDF)
Before this commit: robot panda, 22 links, 21 joints
Links:
- added link panda_ball
Joints:
- added joint panda_tcp_ball_joint: type fixed, parent panda_hand_tcp, child panda_ball, origin xyz=0 0 0.1284 rpy=0 0 0
- joint panda_hand_tcp_joint: origin xyz=0 0 0.1284 rpy=0 0 0 -> xyz=0 0 0.1034 rpy=0 0 0

Commit message: Working CLI and added some default robots for iiwa and panda.

File: assets/panda.urdf (robot description, URDF)
Before this commit: robot panda, 23 links, 22 joints
Links:
- removed link panda_ball
- removed link panda_hand_sc
- removed link panda_link0_sc
- removed link panda_link1_sc
- removed link panda_link2_sc
- removed link panda_link3_sc
- removed link panda_link4_sc
- removed link panda_link5_sc
- removed link panda_link6_sc
- removed link panda_link7_sc
- added link ball_link; visual sphere radius=0.005
- link panda_hand: geometry visual mesh filename=./meshes/panda/hand.dae
- link panda_leftfinger: geometry visual mesh filename=./meshes/panda/finger.dae
- link panda_link0: geometry visual mesh filename=./meshes/panda/link0.dae
- link panda_link1: geometry visual mesh filename=./meshes/panda/link1.dae
- link panda_link2: geometry visual mesh filename=./meshes/panda/link2.dae
- link panda_link3: geometry visual mesh filename=./meshes/panda/link3.dae
- link panda_link4: geometry visual mesh filename=./meshes/panda/link4.dae
- link panda_link5: geometry visual mesh filename=./meshes/panda/link5.dae
- link panda_link6: geometry visual mesh filename=./meshes/panda/link6.dae
- link panda_link7: geometry visual mesh filename=./meshes/panda/link7.dae
- link panda_rightfinger: geometry visual mesh filename=./meshes/panda/finger.dae
Joints:
- removed joint panda_hand_sc_joint
- removed joint panda_link0_sc_joint
- removed joint panda_link1_sc_joint
- removed joint panda_link2_sc_joint
- removed joint panda_link3_sc_joint
- removed joint panda_link4_sc_joint
- removed joint panda_link5_sc_joint
- removed joint panda_link6_sc_joint
- removed joint panda_link7_sc_joint
- removed joint panda_tcp_ball_joint
- added joint ball_joint: type fixed, parent panda_hand_tcp, child ball_link, origin xyz=7.773732033005863e-05 -4.214022515884392e-05 0.030128297908475325 rpy=0.0 0.0 0.0
- joint panda_finger_joint1: axis 0 1 0 -> (none); limit lower=0.0 upper=0.04 effort=100 velocity=0.2 -> (none); type prismatic -> fixed
- joint panda_finger_joint2: axis 0 -1 0 -> (none); limit lower=0.0 upper=0.04 effort=100 velocity=0.2 -> (none); mimic joint=panda_finger_joint1 -> (none); type prismatic -> fixed
