Commit message: Alligns root links to be called base_link and makes required argument an optional.

File: assets/iiwa14_epfl.urdf (robot description, URDF)
Before this commit: robot iiwa14, 11 links, 10 joints
Links:
- removed link iiwa_link_0
- added link base_link, mass 5; visual mesh filename=./meshes/iiwa14/link_0.stl
Joints:
- joint joint_a1: parent iiwa_link_0 -> base_link
- joint world_iiwa_joint: child iiwa_link_0 -> base_link

Commit message: Adds iiwa tool joint offset.

File: assets/iiwa14_epfl.urdf (robot description, URDF)
Before this commit: robot iiwa14, 11 links, 10 joints
Joints:
- joint ball_joint: origin xyz=0 0 0.03 rpy=0 0 0 -> xyz=-6.92119286580406e-05 -0.00018859822675517448 0.03542481345977316 rpy=0.0 0.0 0.0
