Commit message: updated the default urdf such that it would work when using it in the human friendly controllers. I also added a line that automatically generates the panda_calibrated.urdf. This is just changing a path. It is important because otherwise the controller then it does not find the mashes.

File: urdf/panda.urdf (robot description, URDF)
Before this commit: robot panda, 14 links, 13 joints
Joints:
- joint panda_finger_joint1: axis (none) -> 0 1 0; limit (none) -> lower=0.0 upper=0.04 effort=100 velocity=0.2; type fixed -> prismatic
- joint panda_finger_joint2: axis (none) -> 0 -1 0; limit (none) -> lower=0.0 upper=0.04 effort=100 velocity=0.2; mimic (none) -> joint=panda_finger_joint1; type fixed -> prismatic
