Commit message: organized the file in the repo

File: urdf/gen3lite.urdf (robot description, URDF)
Before this commit: robot kinova, 16 links, 15 joints
Links:
- link arm_link: geometry collision mesh filename=../meshes/kinova/arm_link.STL; visual mesh filename=../meshes/kinova/arm_link.STL
- link forearm_link: geometry collision mesh filename=../meshes/kinova/forearm_link.STL; visual mesh filename=../meshes/kinova/forearm_link.STL
- link gripper_base_link: geometry collision mesh filename=../meshes/kinova/gripper_base_link.STL; visual mesh filename=../meshes/kinova/gripper_base_link.STL
- link kinova_base_link: geometry collision mesh filename=../meshes/kinova/base_link.STL; visual mesh filename=../meshes/kinova/base_link.STL
- link left_finger_dist_link: geometry collision mesh filename=../meshes/kinova/left_finger_dist_link.STL; visual mesh filename=../meshes/kinova/left_finger_dist_link.STL
- link left_finger_prox_link: geometry collision mesh filename=../meshes/kinova/left_finger_prox_link.STL; visual mesh filename=../meshes/kinova/left_finger_prox_link.STL
- link lower_wrist_link: geometry collision mesh filename=../meshes/kinova/lower_wrist_link.STL; visual mesh filename=../meshes/kinova/lower_wrist_link.STL
- link right_finger_dist_link: geometry collision mesh filename=../meshes/kinova/right_finger_dist_link.STL; visual mesh filename=../meshes/kinova/right_finger_dist_link.STL
- link right_finger_prox_link: geometry collision mesh filename=../meshes/kinova/right_finger_prox_link.STL; visual mesh filename=../meshes/kinova/right_finger_prox_link.STL
- link shoulder_link: geometry collision mesh filename=../meshes/kinova/shoulder_link.STL; visual mesh filename=../meshes/kinova/shoulder_link.STL
- link upper_wrist_link: geometry collision mesh filename=../meshes/kinova/upper_wrist_link.STL; visual mesh filename=../meshes/kinova/upper_wrist_link.STL

File: urdf/iiwa14.urdf (robot description, URDF)
Before this commit: robot iiwa14, 11 links, 10 joints
Links:
- link base_link: geometry visual mesh filename=../meshes/iiwa14/base_link.dae
- link link_1: geometry visual mesh filename=../meshes/iiwa14/link_1.dae
- link link_2: geometry visual mesh filename=../meshes/iiwa14/link_2.dae
- link link_3: geometry visual mesh filename=../meshes/iiwa14/link_3.dae
- link link_4: geometry visual mesh filename=../meshes/iiwa14/link_4.dae
- link link_5: geometry visual mesh filename=../meshes/iiwa14/link_5.dae
- link link_6: geometry visual mesh filename=../meshes/iiwa14/link_6.dae
- link link_7: geometry visual mesh filename=../meshes/iiwa14/link_7.dae

File: urdf/iiwa14_epfl.urdf (robot description, URDF)
Before this commit: robot iiwa14, 11 links, 10 joints
Links:
- link base_link: geometry visual mesh filename=../meshes/iiwa14/link_0.stl
- link iiwa_link_1: geometry visual mesh filename=../meshes/iiwa14/link_1.stl
- link iiwa_link_2: geometry visual mesh filename=../meshes/iiwa14/link_2.stl
- link iiwa_link_3: geometry visual mesh filename=../meshes/iiwa14/link_3.stl
- link iiwa_link_4: geometry visual mesh filename=../meshes/iiwa14/link_4.stl
- link iiwa_link_5: geometry visual mesh filename=../meshes/iiwa14/link_5.stl
- link iiwa_link_6: geometry visual mesh filename=../meshes/iiwa14/link_6.stl
- link iiwa_link_7: geometry visual mesh filename=../meshes/iiwa14/link_7.stl

File: urdf/panda.urdf (robot description, URDF)
Before this commit: robot panda, 14 links, 13 joints
Links:
- link panda_hand: geometry visual mesh filename=../meshes/panda/hand.dae
- link panda_leftfinger: geometry visual mesh filename=../meshes/panda/finger.dae
- link panda_link0: geometry visual mesh filename=../meshes/panda/link0.dae
- link panda_link1: geometry visual mesh filename=../meshes/panda/link1.dae
- link panda_link2: geometry visual mesh filename=../meshes/panda/link2.dae
- link panda_link3: geometry visual mesh filename=../meshes/panda/link3.dae
- link panda_link4: geometry visual mesh filename=../meshes/panda/link4.dae
- link panda_link5: geometry visual mesh filename=../meshes/panda/link5.dae
- link panda_link6: geometry visual mesh filename=../meshes/panda/link6.dae
- link panda_link7: geometry visual mesh filename=../meshes/panda/link7.dae
- link panda_rightfinger: geometry visual mesh filename=../meshes/panda/finger.dae

File: urdf/vx300s.urdf (robot description, URDF)
Before this commit: robot vx300s, 15 links, 14 joints
Links:
- link base_link: geometry visual mesh filename=../meshes/viper/vx300s_1_base.stl scale=0.001 0.001 0.001
- link gripper_bar_link: geometry visual mesh filename=../meshes/viper/vx300s_9_gripper_bar.stl scale=0.001 0.001 0.001
- link gripper_link: geometry visual mesh filename=../meshes/viper/vx300s_7_gripper.stl scale=0.001 0.001 0.001
- link gripper_prop_link: geometry visual mesh filename=../meshes/viper/vx300s_8_gripper_prop.stl scale=0.001 0.001 0.001
- link left_finger_link: geometry visual mesh filename=../meshes/viper/vx300s_10_gripper_finger.stl scale=0.001 0.001 0.001
- link lower_forearm_link: geometry visual mesh filename=../meshes/viper/vx300s_5_lower_forearm.stl scale=0.001 0.001 0.001
- link right_finger_link: geometry visual mesh filename=../meshes/viper/vx300s_10_gripper_finger.stl scale=0.001 0.001 0.001
- link shoulder_link: geometry visual mesh filename=../meshes/viper/vx300s_2_shoulder.stl scale=0.001 0.001 0.001
- link upper_arm_link: geometry visual mesh filename=../meshes/viper/vx300s_3_upper_arm.stl scale=0.001 0.001 0.001
- link upper_forearm_link: geometry visual mesh filename=../meshes/viper/vx300s_4_upper_forearm.stl scale=0.001 0.001 0.001
- link wrist_link: geometry visual mesh filename=../meshes/viper/vx300s_6_wrist.stl scale=0.001 0.001 0.001

Commit message: updated the nominal models with the right initialization of the the last link

File: urdf/gen3lite.urdf (robot description, URDF)
Before this commit: robot kinova, 16 links, 15 joints
Joints:
- joint ball_joint: origin xyz=0 0 0.17 rpy=0.0 0.0 0.0 -> xyz=0.00038860649894460975 -0.0005822849938650045 0.180196205872143 rpy=0.0 0.0 0.0

File: urdf/iiwa14.urdf (robot description, URDF)
Before this commit: robot iiwa14, 11 links, 10 joints
Joints:
- joint ball_joint: origin xyz=0 0 0.03 rpy=0 0 0 -> xyz=0 0 0.04 rpy=0 0 0
