Commit message: updated README about how to use the calibrated model for the panda, added the calibrated urdf for possible future data analysis, removed some passwords from config files, and delated some corrupted data

File: calibrated_urdf/panda_2/panda.urdf (robot description, URDF)
Before this commit: robot panda, 14 links, 13 joints
Joints:
- joint ball_joint: origin xyz=-0.0009106525430812897 -0.007175258660771381 0.03153248671093189 rpy=0.0 0.0 0.0 -> xyz=0.00037990524928465026 -4.420572608777121e-05 0.03102464075322382 rpy=0.0 0.0 0.0
- joint panda_joint1: origin xyz=-1.2935729674675946e-16 -5.696929452271708e-17 0.33300000000000024 rpy=-2.0355694699737142e-05 -2.8551892429784928e-09 -1.9030793271206534e-17 -> xyz=-1.2758753865242616e-16 -5.2222054042510136e-17 0.333 rpy=8.366805516041043e-06 8.814350308898128e-08 2.4513630387076608e-17
- joint panda_joint2: origin xyz=-0.00014805410119581621 -0.000619168563806805 3.408154257294014e-16 rpy=-1.5663717086115247 0.0009238417600107593 1.0179914805434003e-09 -> xyz=-0.00019417564815309772 -0.00018772077543271004 1.796911857934499e-17 rpy=-1.5725347107345484 0.0009255042963167639 -2.2321032908662564e-15
- joint panda_joint3: origin xyz=0.0003181249935433959 -0.3168341251832623 -0.0006191649945068513 rpy=1.5712448573265205 0.0003675422370507598 0.0008233251486740604 -> xyz=0.0003371033096498455 -0.31626505724737547 -0.0001877201793910496 rpy=1.5720487481374692 0.00011271550591184526 0.0008189810488676046
- joint panda_joint4: origin xyz=0.08199831437787787 0.0001957222099840283 0.0008346641993008366 rpy=1.568597543632454 0.0017324032007747278 -0.0003840582655969283 -> xyz=0.08250428687456778 -0.0002847200612681194 0.0002655680887159182 rpy=1.5741434757926136 0.011776708120902118 -9.025189862699405e-05
- joint panda_joint5: origin xyz=-0.08204015585311616 0.38471576074779346 -0.00019369445893610058 rpy=-1.5706033289126102 0.011486580301602819 -0.0014976198095413764 -> xyz=-0.07866941844576122 0.38493907517903264 0.000283829074942361 rpy=-1.569359416779495 0.005129171736623614 -0.01022805489571219
- joint panda_joint6: origin xyz=0.0009333764668138829 3.071152125803715e-05 0.0007164117085875597 rpy=1.567657121829646 0.002087243828705672 0.01148628749964703 -> xyz=0.0006537446895798644 -1.275492785867517e-05 0.0009786397273711831 rpy=1.5705258868617893 -0.00043533480446275005 0.005114480048959338
- joint panda_joint7: origin xyz=0.0886512928565176 -0.0014051767694575263 -1.7728949732386956e-05 rpy=1.5734147361596689 5.659518976060473e-06 -0.0019275003148919855 -> xyz=0.0902493646325364 -0.0008951821978016663 1.636289653042385e-05 rpy=1.5707208785930096 2.6320186308338895e-08 0.0005154940135814471

File: calibrated_urdf/panda_2/panda_calibrated.urdf (robot description, URDF)
Before this commit: robot panda, 14 links, 13 joints
Links:
- link panda_hand: geometry visual mesh filename=package://franka_description/meshes/visual/hand.dae
- link panda_leftfinger: geometry visual mesh filename=package://franka_description/meshes/visual/finger.dae
- link panda_link0: geometry visual mesh filename=package://franka_description/meshes/visual/link0.dae
- link panda_link1: geometry visual mesh filename=package://franka_description/meshes/visual/link1.dae
- link panda_link2: geometry visual mesh filename=package://franka_description/meshes/visual/link2.dae
- link panda_link3: geometry visual mesh filename=package://franka_description/meshes/visual/link3.dae
- link panda_link4: geometry visual mesh filename=package://franka_description/meshes/visual/link4.dae
- link panda_link5: geometry visual mesh filename=package://franka_description/meshes/visual/link5.dae
- link panda_link6: geometry visual mesh filename=package://franka_description/meshes/visual/link6.dae
- link panda_link7: geometry visual mesh filename=package://franka_description/meshes/visual/link7.dae
- link panda_rightfinger: geometry visual mesh filename=package://franka_description/meshes/visual/finger.dae
Joints:
- joint ball_joint: origin xyz=-0.0009106525430812897 -0.007175258660771381 0.03153248671093189 rpy=0.0 0.0 0.0 -> xyz=0.00037990524928465026 -4.420572608777121e-05 0.03102464075322382 rpy=0.0 0.0 0.0
- joint panda_joint1: origin xyz=-1.2935729674675946e-16 -5.696929452271708e-17 0.33300000000000024 rpy=-2.0355694699737142e-05 -2.8551892429784928e-09 -1.9030793271206534e-17 -> xyz=-1.2758753865242616e-16 -5.2222054042510136e-17 0.333 rpy=8.366805516041043e-06 8.814350308898128e-08 2.4513630387076608e-17
- joint panda_joint2: origin xyz=-0.00014805410119581621 -0.000619168563806805 3.408154257294014e-16 rpy=-1.5663717086115247 0.0009238417600107593 1.0179914805434003e-09 -> xyz=-0.00019417564815309772 -0.00018772077543271004 1.796911857934499e-17 rpy=-1.5725347107345484 0.0009255042963167639 -2.2321032908662564e-15
- joint panda_joint3: origin xyz=0.0003181249935433959 -0.3168341251832623 -0.0006191649945068513 rpy=1.5712448573265205 0.0003675422370507598 0.0008233251486740604 -> xyz=0.0003371033096498455 -0.31626505724737547 -0.0001877201793910496 rpy=1.5720487481374692 0.00011271550591184526 0.0008189810488676046
- joint panda_joint4: origin xyz=0.08199831437787787 0.0001957222099840283 0.0008346641993008366 rpy=1.568597543632454 0.0017324032007747278 -0.0003840582655969283 -> xyz=0.08250428687456778 -0.0002847200612681194 0.0002655680887159182 rpy=1.5741434757926136 0.011776708120902118 -9.025189862699405e-05
- joint panda_joint5: origin xyz=-0.08204015585311616 0.38471576074779346 -0.00019369445893610058 rpy=-1.5706033289126102 0.011486580301602819 -0.0014976198095413764 -> xyz=-0.07866941844576122 0.38493907517903264 0.000283829074942361 rpy=-1.569359416779495 0.005129171736623614 -0.01022805489571219
- joint panda_joint6: origin xyz=0.0009333764668138829 3.071152125803715e-05 0.0007164117085875597 rpy=1.567657121829646 0.002087243828705672 0.01148628749964703 -> xyz=0.0006537446895798644 -1.275492785867517e-05 0.0009786397273711831 rpy=1.5705258868617893 -0.00043533480446275005 0.005114480048959338
- joint panda_joint7: origin xyz=0.0886512928565176 -0.0014051767694575263 -1.7728949732386956e-05 rpy=1.5734147361596689 5.659518976060473e-06 -0.0019275003148919855 -> xyz=0.0902493646325364 -0.0008951821978016663 1.636289653042385e-05 rpy=1.5707208785930096 2.6320186308338895e-08 0.0005154940135814471

File: calibrated_urdf/panda_3/panda.urdf (robot description, URDF)
Before this commit: robot panda, 14 links, 13 joints
Joints:
- joint ball_joint: origin xyz=-0.0009106525430812897 -0.007175258660771381 0.03153248671093189 rpy=0.0 0.0 0.0 -> xyz=0.0003778447912426314 0.00017972692094397734 0.031091389390698887 rpy=0.0 0.0 0.0
- joint panda_joint1: origin xyz=-1.2935729674675946e-16 -5.696929452271708e-17 0.33300000000000024 rpy=-2.0355694699737142e-05 -2.8551892429784928e-09 -1.9030793271206534e-17 -> xyz=-4.718650895518294e-17 1.8269338078033916e-17 0.3330000000000001 rpy=1.443060036170693e-06 -1.1141116109698583e-08 4.155029228558349e-17
- joint panda_joint2: origin xyz=-0.00014805410119581621 -0.000619168563806805 3.408154257294014e-16 rpy=-1.5663717086115247 0.0009238417600107593 1.0179914805434003e-09 -> xyz=-0.00030272394705944304 0.0001314392452688879 9.108197157677059e-17 rpy=-1.569224519569118 0.00025953051430076826 -1.231885684286843e-12
- joint panda_joint3: origin xyz=0.0003181249935433959 -0.3168341251832623 -0.0006191649945068513 rpy=1.5712448573265205 0.0003675422370507598 0.0008233251486740604 -> xyz=0.0002806590580034444 -0.31598109159365023 0.0001314389571123128 rpy=1.5699519202736834 0.0001772122188351117 0.000170842570736644
- joint panda_joint4: origin xyz=0.08199831437787787 0.0001957222099840283 0.0008346641993008366 rpy=1.568597543632454 0.0017324032007747278 -0.0003840582655969283 -> xyz=0.0821772511639403 -5.357729068531642e-05 -1.874942118968558e-05 rpy=1.570329238798954 0.003634167542939902 -0.0001726478966157702
- joint panda_joint5: origin xyz=-0.08204015585311616 0.38471576074779346 -0.00019369445893610058 rpy=-1.5706033289126102 0.011486580301602819 -0.0014976198095413764 -> xyz=-0.08166184278074558 0.38416878967114904 5.362369925985596e-05 rpy=-1.5704333701293198 0.0014558181290433314 -0.0032984710877434252
- joint panda_joint6: origin xyz=0.0009333764668138829 3.071152125803715e-05 0.0007164117085875597 rpy=1.567657121829646 0.002087243828705672 0.01148628749964703 -> xyz=-4.8597064810259795e-05 0.0004293227821836948 0.00017157328439707152 rpy=1.567932496342769 0.00015208320336658598 0.0014546210159514484
- joint panda_joint7: origin xyz=0.0886512928565176 -0.0014051767694575263 -1.7728949732386956e-05 rpy=1.5734147361596689 5.659518976060473e-06 -0.0019275003148919855 -> xyz=0.08770649743939672 -0.0009630206421383316 -0.00042889992127301946 rpy=1.5709182503980177 -2.2182325530324566e-08 -6.317227097718112e-05

File: calibrated_urdf/panda_3/panda_calibrated.urdf (robot description, URDF)
Before this commit: robot panda, 14 links, 13 joints
Links:
- link panda_hand: geometry visual mesh filename=package://franka_description/meshes/visual/hand.dae
- link panda_leftfinger: geometry visual mesh filename=package://franka_description/meshes/visual/finger.dae
- link panda_link0: geometry visual mesh filename=package://franka_description/meshes/visual/link0.dae
- link panda_link1: geometry visual mesh filename=package://franka_description/meshes/visual/link1.dae
- link panda_link2: geometry visual mesh filename=package://franka_description/meshes/visual/link2.dae
- link panda_link3: geometry visual mesh filename=package://franka_description/meshes/visual/link3.dae
- link panda_link4: geometry visual mesh filename=package://franka_description/meshes/visual/link4.dae
- link panda_link5: geometry visual mesh filename=package://franka_description/meshes/visual/link5.dae
- link panda_link6: geometry visual mesh filename=package://franka_description/meshes/visual/link6.dae
- link panda_link7: geometry visual mesh filename=package://franka_description/meshes/visual/link7.dae
- link panda_rightfinger: geometry visual mesh filename=package://franka_description/meshes/visual/finger.dae
Joints:
- joint ball_joint: origin xyz=-0.0009106525430812897 -0.007175258660771381 0.03153248671093189 rpy=0.0 0.0 0.0 -> xyz=0.0003778447912426314 0.00017972692094397734 0.031091389390698887 rpy=0.0 0.0 0.0
- joint panda_joint1: origin xyz=-1.2935729674675946e-16 -5.696929452271708e-17 0.33300000000000024 rpy=-2.0355694699737142e-05 -2.8551892429784928e-09 -1.9030793271206534e-17 -> xyz=-4.718650895518294e-17 1.8269338078033916e-17 0.3330000000000001 rpy=1.443060036170693e-06 -1.1141116109698583e-08 4.155029228558349e-17
- joint panda_joint2: origin xyz=-0.00014805410119581621 -0.000619168563806805 3.408154257294014e-16 rpy=-1.5663717086115247 0.0009238417600107593 1.0179914805434003e-09 -> xyz=-0.00030272394705944304 0.0001314392452688879 9.108197157677059e-17 rpy=-1.569224519569118 0.00025953051430076826 -1.231885684286843e-12
- joint panda_joint3: origin xyz=0.0003181249935433959 -0.3168341251832623 -0.0006191649945068513 rpy=1.5712448573265205 0.0003675422370507598 0.0008233251486740604 -> xyz=0.0002806590580034444 -0.31598109159365023 0.0001314389571123128 rpy=1.5699519202736834 0.0001772122188351117 0.000170842570736644
- joint panda_joint4: origin xyz=0.08199831437787787 0.0001957222099840283 0.0008346641993008366 rpy=1.568597543632454 0.0017324032007747278 -0.0003840582655969283 -> xyz=0.0821772511639403 -5.357729068531642e-05 -1.874942118968558e-05 rpy=1.570329238798954 0.003634167542939902 -0.0001726478966157702
- joint panda_joint5: origin xyz=-0.08204015585311616 0.38471576074779346 -0.00019369445893610058 rpy=-1.5706033289126102 0.011486580301602819 -0.0014976198095413764 -> xyz=-0.08166184278074558 0.38416878967114904 5.362369925985596e-05 rpy=-1.5704333701293198 0.0014558181290433314 -0.0032984710877434252
- joint panda_joint6: origin xyz=0.0009333764668138829 3.071152125803715e-05 0.0007164117085875597 rpy=1.567657121829646 0.002087243828705672 0.01148628749964703 -> xyz=-4.8597064810259795e-05 0.0004293227821836948 0.00017157328439707152 rpy=1.567932496342769 0.00015208320336658598 0.0014546210159514484
- joint panda_joint7: origin xyz=0.0886512928565176 -0.0014051767694575263 -1.7728949732386956e-05 rpy=1.5734147361596689 5.659518976060473e-06 -0.0019275003148919855 -> xyz=0.08770649743939672 -0.0009630206421383316 -0.00042889992127301946 rpy=1.5709182503980177 -2.2182325530324566e-08 -6.317227097718112e-05

File: calibrated_urdf/panda_4/panda.urdf (robot description, URDF)
Before this commit: robot panda, 14 links, 13 joints
Joints:
- joint ball_joint: origin xyz=-0.0009106525430812897 -0.007175258660771381 0.03153248671093189 rpy=0.0 0.0 0.0 -> xyz=-0.0009481981012812722 -0.007071742271933424 0.031439169882774995 rpy=0.0 0.0 0.0
- joint panda_joint1: origin xyz=-1.2935729674675946e-16 -5.696929452271708e-17 0.33300000000000024 rpy=-2.0355694699737142e-05 -2.8551892429784928e-09 -1.9030793271206534e-17 -> xyz=5.774688145414098e-17 2.218661989219751e-17 0.333 rpy=-6.478369884611035e-06 3.2531259337282877e-08 -3.351756093527367e-17
- joint panda_joint2: origin xyz=-0.00014805410119581621 -0.000619168563806805 3.408154257294014e-16 rpy=-1.5663717086115247 0.0009238417600107593 1.0179914805434003e-09 -> xyz=6.869792075033197e-05 0.00019688359843828975 -2.1505593657772702e-17 rpy=-1.5691039237056728 0.0004677993350039688 1.4241498262028565e-10
- joint panda_joint3: origin xyz=0.0003181249935433959 -0.3168341251832623 -0.0006191649945068513 rpy=1.5712448573265205 0.0003675422370507598 0.0008233251486740604 -> xyz=4.4999344066411925e-05 -0.3168198111414633 0.00019688348264730338 rpy=1.569905108582915 -0.0026702643847938334 0.00045357944186582064
- joint panda_joint4: origin xyz=0.08199831437787787 0.0001957222099840283 0.0008346641993008366 rpy=1.568597543632454 0.0017324032007747278 -0.0003840582655969283 -> xyz=0.08265427273481392 0.0002036643475814555 0.0008200064152495127 rpy=1.5691394826589014 0.0013927386555089988 0.0026538673212457547
- joint panda_joint5: origin xyz=-0.08204015585311616 0.38471576074779346 -0.00019369445893610058 rpy=-1.5706033289126102 0.011486580301602819 -0.0014976198095413764 -> xyz=-0.08204134414108213 0.3847534044806093 -0.00020189521090589624 rpy=-1.5716993777741444 0.011030878222247893 -0.0011500632899242276
- joint panda_joint6: origin xyz=0.0009333764668138829 3.071152125803715e-05 0.0007164117085875597 rpy=1.567657121829646 0.002087243828705672 0.01148628749964703 -> xyz=0.0008069285645448682 0.0006930431259015023 0.0007541089343999483 rpy=1.565906533038832 0.002447279527486587 0.011031931752826084
- joint panda_joint7: origin xyz=0.0886512928565176 -0.0014051767694575263 -1.7728949732386956e-05 rpy=1.5734147361596689 5.659518976060473e-06 -0.0019275003148919855 -> xyz=0.08789623448965604 -0.0013118880147136493 -0.0006803956263812915 rpy=1.569037177169469 -3.4146334876909247e-06 -0.002277927431706217

File: calibrated_urdf/panda_4/panda_calibrated.urdf (robot description, URDF)
Before this commit: robot panda, 14 links, 13 joints
Links:
- link panda_hand: geometry visual mesh filename=package://franka_description/meshes/visual/hand.dae
- link panda_leftfinger: geometry visual mesh filename=package://franka_description/meshes/visual/finger.dae
- link panda_link0: geometry visual mesh filename=package://franka_description/meshes/visual/link0.dae
- link panda_link1: geometry visual mesh filename=package://franka_description/meshes/visual/link1.dae
- link panda_link2: geometry visual mesh filename=package://franka_description/meshes/visual/link2.dae
- link panda_link3: geometry visual mesh filename=package://franka_description/meshes/visual/link3.dae
- link panda_link4: geometry visual mesh filename=package://franka_description/meshes/visual/link4.dae
- link panda_link5: geometry visual mesh filename=package://franka_description/meshes/visual/link5.dae
- link panda_link6: geometry visual mesh filename=package://franka_description/meshes/visual/link6.dae
- link panda_link7: geometry visual mesh filename=package://franka_description/meshes/visual/link7.dae
- link panda_rightfinger: geometry visual mesh filename=package://franka_description/meshes/visual/finger.dae
Joints:
- joint ball_joint: origin xyz=-0.0009106525430812897 -0.007175258660771381 0.03153248671093189 rpy=0.0 0.0 0.0 -> xyz=-0.0009481981012812722 -0.007071742271933424 0.031439169882774995 rpy=0.0 0.0 0.0
- joint panda_joint1: origin xyz=-1.2935729674675946e-16 -5.696929452271708e-17 0.33300000000000024 rpy=-2.0355694699737142e-05 -2.8551892429784928e-09 -1.9030793271206534e-17 -> xyz=5.774688145414098e-17 2.218661989219751e-17 0.333 rpy=-6.478369884611035e-06 3.2531259337282877e-08 -3.351756093527367e-17
- joint panda_joint2: origin xyz=-0.00014805410119581621 -0.000619168563806805 3.408154257294014e-16 rpy=-1.5663717086115247 0.0009238417600107593 1.0179914805434003e-09 -> xyz=6.869792075033197e-05 0.00019688359843828975 -2.1505593657772702e-17 rpy=-1.5691039237056728 0.0004677993350039688 1.4241498262028565e-10
- joint panda_joint3: origin xyz=0.0003181249935433959 -0.3168341251832623 -0.0006191649945068513 rpy=1.5712448573265205 0.0003675422370507598 0.0008233251486740604 -> xyz=4.4999344066411925e-05 -0.3168198111414633 0.00019688348264730338 rpy=1.569905108582915 -0.0026702643847938334 0.00045357944186582064
- joint panda_joint4: origin xyz=0.08199831437787787 0.0001957222099840283 0.0008346641993008366 rpy=1.568597543632454 0.0017324032007747278 -0.0003840582655969283 -> xyz=0.08265427273481392 0.0002036643475814555 0.0008200064152495127 rpy=1.5691394826589014 0.0013927386555089988 0.0026538673212457547
- joint panda_joint5: origin xyz=-0.08204015585311616 0.38471576074779346 -0.00019369445893610058 rpy=-1.5706033289126102 0.011486580301602819 -0.0014976198095413764 -> xyz=-0.08204134414108213 0.3847534044806093 -0.00020189521090589624 rpy=-1.5716993777741444 0.011030878222247893 -0.0011500632899242276
- joint panda_joint6: origin xyz=0.0009333764668138829 3.071152125803715e-05 0.0007164117085875597 rpy=1.567657121829646 0.002087243828705672 0.01148628749964703 -> xyz=0.0008069285645448682 0.0006930431259015023 0.0007541089343999483 rpy=1.565906533038832 0.002447279527486587 0.011031931752826084
- joint panda_joint7: origin xyz=0.0886512928565176 -0.0014051767694575263 -1.7728949732386956e-05 rpy=1.5734147361596689 5.659518976060473e-06 -0.0019275003148919855 -> xyz=0.08789623448965604 -0.0013118880147136493 -0.0006803956263812915 rpy=1.569037177169469 -3.4146334876909247e-06 -0.002277927431706217

File: calibrated_urdf/panda_6/panda.urdf (robot description, URDF)
Before this commit: robot panda, 14 links, 13 joints
Joints:
- joint panda_finger_joint1: axis (none) -> 0 1 0; limit (none) -> lower=0.0 upper=0.04 effort=100 velocity=0.2; type fixed -> prismatic
- joint panda_finger_joint2: axis (none) -> 0 -1 0; limit (none) -> lower=0.0 upper=0.04 effort=100 velocity=0.2; mimic (none) -> joint=panda_finger_joint1; type fixed -> prismatic

File: calibrated_urdf/panda_6/panda_calibrated.urdf (robot description, URDF)
Before this commit: robot panda, 14 links, 13 joints
Links:
- link panda_hand: geometry visual mesh filename=package://franka_description/meshes/visual/hand.dae
- link panda_leftfinger: geometry visual mesh filename=package://franka_description/meshes/visual/finger.dae
- link panda_link0: geometry visual mesh filename=package://franka_description/meshes/visual/link0.dae
- link panda_link1: geometry visual mesh filename=package://franka_description/meshes/visual/link1.dae
- link panda_link2: geometry visual mesh filename=package://franka_description/meshes/visual/link2.dae
- link panda_link3: geometry visual mesh filename=package://franka_description/meshes/visual/link3.dae
- link panda_link4: geometry visual mesh filename=package://franka_description/meshes/visual/link4.dae
- link panda_link5: geometry visual mesh filename=package://franka_description/meshes/visual/link5.dae
- link panda_link6: geometry visual mesh filename=package://franka_description/meshes/visual/link6.dae
- link panda_link7: geometry visual mesh filename=package://franka_description/meshes/visual/link7.dae
- link panda_rightfinger: geometry visual mesh filename=package://franka_description/meshes/visual/finger.dae
Joints:
- joint ball_joint: origin xyz=-0.0009106525430812897 -0.007175258660771381 0.03153248671093189 rpy=0.0 0.0 0.0 -> xyz=-0.000964425639282203 -0.007034307145014577 0.031774138437114886 rpy=0.0 0.0 0.0
- joint panda_joint1: origin xyz=-1.2935729674675946e-16 -5.696929452271708e-17 0.33300000000000024 rpy=-2.0355694699737142e-05 -2.8551892429784928e-09 -1.9030793271206534e-17 -> xyz=2.4693690209296155e-17 -4.567396885044367e-17 0.3330000000000001 rpy=-2.6313949212650455e-06 -5.186632432689784e-08 -1.2780383157481656e-17
- joint panda_joint2: origin xyz=-0.00014805410119581621 -0.000619168563806805 3.408154257294014e-16 rpy=-1.5663717086115247 0.0009238417600107593 1.0179914805434003e-09 -> xyz=-0.00016542285187714177 0.00046611959924426654 4.3408992507204626e-17 rpy=-1.5671631233681536 -0.0006063905110036522 -4.638746785761078e-16
- joint panda_joint3: origin xyz=0.0003181249935433959 -0.3168341251832623 -0.0006191649945068513 rpy=1.5712448573265205 0.0003675422370507598 0.0008233251486740604 -> xyz=-4.018702287107603e-05 -0.31650707253508886 0.00046611688726827104 rpy=1.5675434452162544 0.007116873693165347 -0.0005936954139923941
- joint panda_joint4: origin xyz=0.08199831437787787 0.0001957222099840283 0.0008346641993008366 rpy=1.568597543632454 0.0017324032007747278 -0.0003840582655969283 -> xyz=0.08298433483169573 -0.0008116166118042272 0.0005086088803250237 rpy=1.5720164890105501 0.001378946498497616 -0.007051884242910425
- joint panda_joint5: origin xyz=-0.08204015585311616 0.38471576074779346 -0.00019369445893610058 rpy=-1.5706033289126102 0.011486580301602819 -0.0014976198095413764 -> xyz=-0.082508298986969 0.38458342771047327 0.000807558975830882 rpy=-1.569984004153357 0.003846076429680107 -0.0013253971011171648
- joint panda_joint6: origin xyz=0.0009333764668138829 3.071152125803715e-05 0.0007164117085875597 rpy=1.567657121829646 0.002087243828705672 0.01148628749964703 -> xyz=-0.00015157481312079457 0.00035924901235692046 0.0005840719712579211 rpy=1.5668251155588273 0.002949000686762804 0.0038450010406930564
- joint panda_joint7: origin xyz=0.0886512928565176 -0.0014051767694575263 -1.7728949732386956e-05 rpy=1.5734147361596689 5.659518976060473e-06 -0.0019275003148919855 -> xyz=0.08620360708606715 -0.0016404761909481107 -0.00035750862524293586 rpy=1.571805285853835 3.401850246877615e-06 -0.002789392698002778
