Commit message: updated README about how to use the calibrated model for the panda, added the calibrated urdf for possible future data analysis, removed some passwords from config files, and delated some corrupted data

File: calibrated_urdf/panda_7/panda_calibrated.urdf (robot description, URDF)
Before this commit: robot panda, 14 links, 13 joints
Links:
- link panda_hand: geometry visual mesh filename=package://franka_description/meshes/visual/hand.dae
- link panda_leftfinger: geometry visual mesh filename=package://franka_description/meshes/visual/finger.dae
- link panda_link0: geometry visual mesh filename=package://franka_description/meshes/visual/link0.dae
- link panda_link1: geometry visual mesh filename=package://franka_description/meshes/visual/link1.dae
- link panda_link2: geometry visual mesh filename=package://franka_description/meshes/visual/link2.dae
- link panda_link3: geometry visual mesh filename=package://franka_description/meshes/visual/link3.dae
- link panda_link4: geometry visual mesh filename=package://franka_description/meshes/visual/link4.dae
- link panda_link5: geometry visual mesh filename=package://franka_description/meshes/visual/link5.dae
- link panda_link6: geometry visual mesh filename=package://franka_description/meshes/visual/link6.dae
- link panda_link7: geometry visual mesh filename=package://franka_description/meshes/visual/link7.dae
- link panda_rightfinger: geometry visual mesh filename=package://franka_description/meshes/visual/finger.dae
